Commit message: Remove venv from tracking

File: Dexter_Sim/Models/Dexter_ER2.urdf (robot description, URDF)
Before this commit: robot Dexter_ER2, 7 links, 6 joints
Links:
- link link5: geometry visual cylinder length=0.085 radius=0.018
Joints:
- joint ee_fixed: origin xyz=0 0 0.02 -> xyz=0 0 0.085
- joint joint2: axis 0 1 0 -> 1 0 0
- joint joint3: axis 0 1 0 -> 1 0 0; origin xyz=0.086 0 0 -> xyz=0 0 0.086
- joint joint4: axis 0 1 0 -> 1 0 0; origin xyz=0.077 0 0 -> xyz=0 0 0.077
- joint joint5: limit (none) -> lower=-3.14 upper=3.14 effort=5 velocity=1; origin xyz=0.085 0 0 -> xyz=0 0 0.085
